Commit message: Clean rover_arm setup and rover_urdf clean up

File: software/ros_packages/rover_urdf/urdf/rover_urdf.xacro (robot description, xacro)
@@ -4,6 +4,21 @@
 -->
 <robot name="rover" xmlns:xacro="https://ros.org/wiki/xacro">
-    <!-- Includes (material libraries, etc) -->
-    <!-- Link Chasis with bogies and tower -->
-    <!-- Link Arm or Scimech-->
-        <!-- Arm option for gripper -->
+    <xacro:macro name="rover" params="name attachment:=arm">
+        <!-- Includes (material libraries, etc) -->
+        <xacro:include filename="$(find rover_arm_urdf)/urdf/rover_arm.urdf.xacro" />
+        <xacro:include filename="rover_body.urdf.xacro"/>
+        <!-- Link Chasis with bogies and tower -->
+        <xacro:rover_body name="rover_body">
+        </xacro:rover_body>
+        <!-- Link Arm or Scimech-->
+        <xacro:if value="${attachment== 'arm'}">
+            <xacro:rover_arm parent="rover_base_origin" >
+                <origin rpy= "0.0 0.0 0.0" xyz="0.175735 0 0.03175"/>
+            </xacro:rover_arm>
+        </xacro:if>
+        <xacro:if value="${attachment == 'science'}">
+        </xacro:if>
+            <!-- Arm option for gripper -->
+    </xacro:macro>
+    <xacro:rover name="rover" attachment="arm"/>
+</robot>
