Commit message: Added cams to urdf

File: software/ros_packages/rover_urdf/urdf/rover2_body.urdf (robot description, URDF)
Before this commit: robot rover, 25 links, 26 joints
Links:
- added link camera1
- added link camera_left_chassis
- added link camera_right_chassis
Joints:
- added joint camera_left_chassis: type fixed, parent base_link, child camera1, origin xyz=0.246 0 0.290 rpy=0 0 0.785
- added joint camera_right_chassis: type fixed, parent base_link, child camera2, origin xyz=-0.246 0 0.290 rpy=0 0 -0.785
