Commit message: Added new tower  to urdf

File: software/ros_packages/rover_urdf/urdf/rover2_body.urdf.xacro (robot description, xacro)
@@ -60,5 +60,5 @@
                 <origin xyz="-0.0 -0.0 -0.0" rpy="0 0 0"/>
                 <geometry>
-                <mesh filename="package://rover_urdf/urdf/stl_files/mr2526-Tower-URDF_Collision-Unsimplified.stl" scale="0.001 0.001 0.001"/>
+                <mesh filename="package://rover_urdf/urdf/stl_files/mr2526-Tower-Teli-URDF_Collision.stl" scale="0.001 0.001 0.001"/>
                 </geometry>
                 <material name="silver"/>
@@ -67,5 +67,5 @@
                 <origin xyz="-0.0 -0.0 -0.0" rpy="0 0 0"/>
                 <geometry>
-                <mesh filename="package://rover_urdf/urdf/stl_files/mr2526-Tower-URDF_Collision-Unsimplified.stl" scale="0.001 0.001 0.001"/>
+                <mesh filename="package://rover_urdf/urdf/stl_files/mr2526-Tower-Teli-URDF_Collision.stl" scale="0.001 0.001 0.001"/>
                 </geometry>
             </collision>
