Commit message: Fixed CMakes and added negative gear ratios lmao

File: software/ros_packages/rover_urdf/ros2_control/rover_body.ros2_control.xacro (robot description, xacro)
@@ -66,5 +66,5 @@
             <joint name="rover_front_left_wheel_joint">
                 <param name="node_id">0</param>
-                <param name="gear_ratio">50</param>
+                <param name="gear_ratio">-50</param>
                 <!-- <command_interface name="position"/> -->
                 <command_interface name="velocity"/>
@@ -76,5 +76,5 @@
             <joint name="rover_middle_left_wheel_joint">
                 <param name="node_id">2</param>
-                <param name="gear_ratio">50</param>
+                <param name="gear_ratio">-50</param>
                 <!-- <command_interface name="position"/> -->
                 <command_interface name="velocity"/>
@@ -86,5 +86,5 @@
             <joint name="rover_back_left_wheel_joint">
                 <param name="node_id">4</param>
-                <param name="gear_ratio">50</param>
+                <param name="gear_ratio">-50</param>
                 <!-- <command_interface name="position"/> -->
                 <command_interface name="velocity"/>

File: software/ros_packages/rover_urdf/urdf/rover2_body.urdf.xacro (robot description, xacro)
@@ -435,5 +435,5 @@
             <parent link="${name}_right_bogie"/>
             <child link="${name}_front_right_wheel"/>
-            <axis xyz="-1.0 -0.0 0.0"/>
+            <axis xyz="1.0 -0.0 0.0"/>
         </joint>
         <joint name="${name}_middle_right_wheel_joint" type="continuous">
@@ -441,5 +441,5 @@
             <parent link="${name}_right_bogie"/>
             <child link="${name}_middle_right_wheel"/>
-            <axis xyz="-1.0 0.0 0.0"/>
+            <axis xyz="1.0 0.0 0.0"/>
         </joint>
         <joint name="${name}_back_right_wheel_joint" type="continuous">
@@ -447,5 +447,5 @@
             <parent link="${name}_rear_bogie"/>
             <child link="${name}_back_right_wheel"/>
-            <axis xyz="-1.0 0.0 0.0"/>
+            <axis xyz="1.0 0.0 0.0"/>
         </joint>
         <gazebo reference="${name}_base_origin">
