Commit message: Fixed time parameterization

File: software/ros_packages/rover_arm_urdf/urdf/rover_arm.urdf (robot description, URDF)
Before this commit: robot rover_arm, 14 links, 13 joints
Joints:
- joint base_joint: limit lower=-1.57079632679 upper=1.57079632679 effort=1000.0 velocity=6.0 -> lower=-1.57079632679 upper=1.57079632679 effort=1000.0 velocity=5.5
- joint elbow_pitch_joint: limit lower=-3.1415926 upper=3.1415926 effort=1000.0 velocity=2.0 -> lower=-3.1415926 upper=3.1415926 effort=1000.0 velocity=5.6
- joint elbow_roll_joint: limit lower=-3.141592653589793 upper=3.141592653589793 effort=1000.0 velocity=6.0 -> lower=-3.141592653589793 upper=3.141592653589793 effort=1000.0 velocity=18.5
- joint shoulder_joint: limit lower=-1.57079632679 upper=1.57079632679 effort=1000.0 velocity=6.0 -> lower=-1.57079632679 upper=1.57079632679 effort=1000.0 velocity=3.5
- joint wrist_pitch_joint: limit lower=-1.57079632679 upper=3.141592653589793 effort=1000.0 velocity=6.0 -> lower=-1.57079632679 upper=3.141592653589793 effort=1000.0 velocity=5.9
- joint wrist_roll_joint: limit effort=1000.0 velocity=60.0 -> effort=1000.0 velocity=22.0

Commit message: localization in 3d for proper pitch

File: software/ros_packages/rover_arm_urdf/urdf/rover_arm.urdf (robot description, URDF)
Before this commit: robot rover_arm, 11 links, 10 joints
Joints:
- joint imu_joint: origin xyz=.1524 .1016 0 rpy=0 0 -1.5708 -> xyz=.1524 .1016 0 rpy=-0.0556722 0.116731 -1.5708
