Commit message: Inertias as per Ungrounded URDF exported (may not line up with stl's)

File: software/ros_packages/rover_arm_urdf/urdf/rover2_arm.urdf.xacro (robot description, xacro)
@@ -6,7 +6,7 @@
     <link name="${name}_base_link">
       <inertial>
-        <origin xyz="-0.0009447828005189041 0.08468497648772827 0.03949082514116446" rpy="0 0 0"/>
+        <origin xyz="0.08371 -0.000083675 0.03944" rpy="0 0 -1.5708"/>
         <mass value="1.9803212654096218"/>
-        <inertia ixx="0.003733" iyy="0.007147" izz="0.007072" ixy="1e-06" iyz="-3e-06" ixz="0.001344"/>
+        <inertia ixx="0.003734" iyy="0.007149" izz="0.007073" ixy="1.085e-06" iyz="-3.675e-06" ixz="0.001344"/>
       </inertial>
       <visual>
@@ -26,7 +26,7 @@
     <link name="${name}_shoulder">
       <inertial>
-        <origin xyz="-0.0005179666729459471 -0.009703141635556661 0.11413506870321072" rpy="0 0 0"/>
+        <origin xyz="0.0094258 0.0003306 0.11444" rpy="0 0 0"/>
         <mass value="4.597426515663195"/>
-        <inertia ixx="0.034023" iyy="0.017924" izz="0.026762" ixy="-0.000625" iyz="-0.000848" ixz="-1e-05"/>
+        <inertia ixx="0.017924" iyy="0.03421" izz="0.026905" ixy="0.000571" iyz="3.3e-05" ixz="0.000896"/>
       </inertial>
       <visual>
@@ -46,7 +46,7 @@
     <link name="${name}_long_arm">
       <inertial>
-        <origin xyz="0.003255341560779442 0.08225313572805198 0.3038514362100365" rpy="0 0 0"/>
+        <origin xyz="-0.082265 -0.002920 0.304191" rpy="0 0 0"/>
         <mass value="1.931219575863863"/>
-        <inertia ixx="0.103823" iyy="0.102679" izz="0.003018" ixy="-4.5e-05" iyz="-0.00607" ixz="-0.00024"/>
+        <inertia ixx="0.102866" iyy="0.10401" izz="0.003018" ixy="-4.1e-05" iyz="0.00216" ixz="0.006075"/>
       </inertial>
       <visual>
@@ -66,7 +66,7 @@
     <link name="${name}_elbow_roll">
       <inertial>
-        <origin xyz="0.0028418040335443616 0.062929193683773 0.002447775776976968" rpy="0 0 0"/>
+        <origin xyz="0.06296 -0.001884  0.002448" rpy="0 0 0"/>
         <mass value="1.6182387209715599"/>
-        <inertia ixx="0.002773" iyy="0.002583" izz="0.001869" ixy="-9e-06" iyz="-1e-05" ixz="3.1e-05"/>
+        <inertia ixx="0.002582" iyy="0.002773" izz="0.001869" ixy="-5e-06" iyz="3.2e-05" ixz="7e-05"/>
       </inertial>
       <visual>
@@ -86,7 +86,7 @@
     <link name="${name}_short_arm">
       <inertial>
-        <origin xyz="0.0008005407654101404 0.019869467859255252 0.3086627160724952" rpy="0 0 0"/>
+        <origin xyz="-0.019578 -0.0008965 0.308656" rpy="0 0 0"/>
         <mass value="2.3532339025644338"/>
-        <inertia ixx="0.029335" iyy="0.024849" izz="0.007089" ixy="-0.000181" iyz="-0.001871" ixz="-7.4e-05"/>
+        <inertia ixx="0.024841" iyy="0.029375" izz="0.007124" ixy="-0.000127" iyz="8.7e-05" ixz="0.001874"/>
       </inertial>
       <visual>
@@ -106,7 +106,7 @@
     <link name="${name}_wrist_roll">
       <inertial>
-        <origin xyz="-0.08875188207831092 -0.016654911934429514 -0.03711756226850449" rpy="0 0 0"/>
+        <origin xyz="0.048557 0.002168 -0.03599" rpy="0 0 0"/>
         <mass value="1.3442681899530171"/>
-        <inertia ixx="0.002669" iyy="0.002554" izz="0.00167" ixy="-1.6e-05" iyz="-8.4e-05" ixz="-9e-06"/>
+        <inertia ixx="0.002484" iyy="0.002597" izz="0.001636" ixy="8e-06" iyz="4.8e-05" ixz="8.1e-05"/>
       </inertial>
       <visual>
@@ -126,7 +126,7 @@
     <link name="${name}_tool0">
       <inertial>
-        <origin xyz="4.7031710182124375e-05 0.000453106103411427 0.01635440962044843" rpy="0 0 0"/>
+        <origin xyz="-0.00042542 0.00016296 0.016355" rpy="0 0 0"/>
         <mass value="0.09744608224670866"/>
-        <inertia ixx="3.3e-05" iyy="3.4e-05" izz="5.6e-05" ixy="0.0" iyz="-0.0" ixz="-0.0"/>
+        <inertia ixx="3.3e-05" iyy="3.3e-05" izz="5.6e-05" ixy="0.0" iyz="0.0" ixz="0.0"/>
       </inertial>
       <visual>
@@ -146,7 +146,7 @@
     <link name="${name}_gripper">
       <inertial>
-        <origin xyz="-0.0034288329615621872 4.165532799299543e-05 0.09155079805740618" rpy="0 0 0"/>
+        <origin xyz="0.00054881 -0.003385 0.09155" rpy="0 0 0"/>
         <mass value="1.436142089281915"/>
-        <inertia ixx="0.00626" iyy="0.004291" izz="0.003365" ixy="-0.000241" iyz="-0.000136" ixz="8e-05"/>
+        <inertia ixx="0.004268" iyy="0.006284" izz="0.003365" ixy="-0.000106" iyz="0.000102" ixz="0.00012"/>
       </inertial>
       <visual>

Commit message: moving rover ish

File: software/ros_packages/rover_arm_urdf/urdf/rover2_arm.urdf.xacro (robot description, xacro)
@@ -182,5 +182,5 @@
       <child link="${name}_shoulder"/>
       <axis xyz="0.0 0.0 -1.0"/>
-      <limit upper="1.570796" lower="-1.570796" effort="100" velocity="100"/>
+      <limit upper="1.570796" lower="-1.570796" effort="100" velocity="0.565478"/>
     </joint>
     <joint name="${name}_shoulder_joint" type="revolute">
@@ -189,5 +189,5 @@
       <child link="${name}_long_arm"/>
       <axis xyz="1.0 0.0 0.0"/>
-      <limit upper="1.570796" lower="-1.570796" effort="100" velocity="100"/>
+      <limit upper="1.570796" lower="-1.570796" effort="100" velocity="0.353429"/>
     </joint>
     <joint name="${name}_elbow_pitch_joint" type="revolute">
@@ -196,5 +196,5 @@
       <child link="${name}_elbow_roll"/>
       <axis xyz="1.0 0.0 0.0"/>
-      <limit upper="3.141593" lower="-3.141593" effort="100" velocity="100"/>
+      <limit upper="3.141593" lower="-3.141593" effort="100" velocity="0.604799"/>
     </joint>
     <joint name="${name}_elbow_roll_joint" type="revolute">
@@ -203,5 +203,5 @@
       <child link="${name}_short_arm"/>
       <axis xyz="0.0 0.0 -1.0"/>
-      <limit upper="3.141593" lower="-3.141593" effort="100" velocity="100"/>
+      <limit upper="3.141593" lower="-3.141593" effort="100" velocity="1.884956"/>
     </joint>
     <joint name="${name}_wrist_pitch_joint" type="revolute">
@@ -210,5 +210,5 @@
       <child link="${name}_wrist_roll"/>
       <axis xyz="1.0 0.0 0.0"/>
-      <limit upper="3.141593" lower="-3.141593" effort="100" velocity="100"/>
+      <limit upper="3.141593" lower="-3.141593" effort="100" velocity="0.611337"/>
     </joint>
     <joint name="${name}_wrist_roll_joint" type="continuous">
@@ -217,4 +217,5 @@
       <child link="${name}_tool0"/>
       <axis xyz="0.0 0.0 1.0"/>
+      <limit effort="100" velocity="2.261947"/>
     </joint>
     <joint name="${name}_gripper_joint" type="fixed">
