Commit message: Working nav2 stack teli-op

File: software/ros_packages/rover2_arm/config/rover.urdf.xacro (robot description, xacro)
@@ -9,5 +9,5 @@
     <!-- Import rover urdf file -->
     <xacro:include filename="$(find rover_urdf)/urdf/rover2_urdf.xacro" />
-    <xacro:rover name="rover" attachment="$(arg attachment)"/>
+    <xacro:rover name="rover" attachment="$(arg attachment)" hardware_type="(arg ros2_control_hardware_type)"/>
     <!-- Import control_xacro -->
     <xacro:include filename="rover.ros2_control.xacro" />

File: software/ros_packages/rover_urdf/ros2_control/rover_body.ros2_control.xacro (robot description, xacro)
@@ -8,5 +8,4 @@
                     <plugin>odrive_ros2_control_plugin/ODriveHardwareInterface</plugin>
                     <param name="can">can0</param>
-                    <plugin>mock_components/GenericSystem</plugin>
                 </xacro:if>
                 <xacro:if value="${ros2_control_hardware_type == 'sim'}">
@@ -17,51 +16,4 @@
                 </xacro:if>
             </hardware>
-            <!-- <joint name="rover_front_left_link_joint">
-                <state_interface name="position">
-                    <param name="initial_value">${initial_positions['rover_front_left_link_joint']}</param>
-                </state_interface>
-            </joint>
-            <joint name="rover_back_left_link_joint">
-                <state_interface name="position">
-                    <param name="initial_value">${initial_positions['rover_back_left_link_joint']}</param>
-                </state_interface>
-            </joint>
-            <joint name="rover_front_left_bogie_joint">
-                <state_interface name="position">
-                    <param name="initial_value">${initial_positions['rover_front_left_bogie_joint']}</param>
-                </state_interface>
-            </joint> -->
-            <!-- Four Bar linkage doesn't exist in URDF's -->
-            <!-- <joint name="rover_back_left_bogie_joint">
-                <state_interface name="position">
-                    <param name="initial_value">${initial_positions['rover_back_left_bogie_joint']}</param>
-                </state_interface>
-            </joint> -->
-            <!--<joint name="rover_front_right_link_joint">
-                <state_interface name="position">
-                    <param name="initial_value">${initial_positions['rover_front_right_link_joint']}</param>
-                </state_interface>
-            </joint>
-            <joint name="rover_back_right_link_joint">
-                <state_interface name="position">
-                    <param name="initial_value">${initial_positions['rover_back_right_link_joint']}</param>
-                </state_interface>
-            </joint>
-            <joint name="rover_front_right_bogie_joint">
-                <state_interface name="position">
-                    <param name="initial_value">${initial_positions['rover_front_right_bogie_joint']}</param>
-                </state_interface>
-            </joint>-->
-            <!-- Four Bar linkage doesn't exist in URDF's -->
-            <!-- <joint name="rover_back_right_bogie_joint">
-                <state_interface name="position">
-                    <param name="initial_value">${initial_positions['rover_back_right_bogie_joint']}</param>
-                </state_interface>
-            </joint> -->
-            <!--<joint name="rover_rear_bogie_joint">
-                <state_interface name="position">
-                    <param name="initial_value">${initial_positions['rover_rear_bogie_joint']}</param>
-                </state_interface>
-            </joint>-->
             <joint name="rover_front_left_wheel_joint">
                 <param name="node_id">0</param>
@@ -125,4 +77,64 @@
             </joint>
         </ros2_control>
+        <ros2_control  name="${name}_passive" type="system">
+            <hardware>
+                <xacro:if value="${ros2_control_hardware_type == 'main'}">
+                    <plugin>mock_components/GenericSystem</plugin>
+                </xacro:if>
+                <xacro:if value="${ros2_control_hardware_type == 'sim'}">
+                    <plugin>mock_components/GenericSystem</plugin>
+                </xacro:if>
+                <xacro:if value="${ros2_control_hardware_type == 'gazebo'}">
+                    <plugin>gz_ros2_control/GazeboSimSystem</plugin>
+                </xacro:if>
+            </hardware>
+            <joint name="rover_front_left_link_joint">
+                <state_interface name="position">
+                    <param name="initial_value">${initial_positions['rover_front_left_link_joint']}</param>
+                </state_interface>
+            </joint>
+            <joint name="rover_back_left_link_joint">
+                <state_interface name="position">
+                    <param name="initial_value">${initial_positions['rover_back_left_link_joint']}</param>
+                </state_interface>
+            </joint>
+            <joint name="rover_front_left_bogie_joint">
+                <state_interface name="position">
+                    <param name="initial_value">${initial_positions['rover_front_left_bogie_joint']}</param>
+                </state_interface>
+            </joint>
+            <!-- Four Bar linkage doesn't exist in URDF's -->
+            <!-- <joint name="rover_back_left_bogie_joint">
+                <state_interface name="position">
+                    <param name="initial_value">${initial_positions['rover_back_left_bogie_joint']}</param>
+                </state_interface>
+            </joint> -->
+            <joint name="rover_front_right_link_joint">
+                <state_interface name="position">
+                    <param name="initial_value">${initial_positions['rover_front_right_link_joint']}</param>
+                </state_interface>
+            </joint>
+            <joint name="rover_back_right_link_joint">
+                <state_interface name="position">
+                    <param name="initial_value">${initial_positions['rover_back_right_link_joint']}</param>
+                </state_interface>
+            </joint>
+            <joint name="rover_front_right_bogie_joint">
+                <state_interface name="position">
+                    <param name="initial_value">${initial_positions['rover_front_right_bogie_joint']}</param>
+                </state_interface>
+            </joint>
+            <!-- Four Bar linkage doesn't exist in URDF's -->
+            <!-- <joint name="rover_back_right_bogie_joint">
+                <state_interface name="position">
+                    <param name="initial_value">${initial_positions['rover_back_right_bogie_joint']}</param>
+                </state_interface>
+            </joint> -->
+            <joint name="rover_rear_bogie_joint">
+                <state_interface name="position">
+                    <param name="initial_value">${initial_positions['rover_rear_bogie_joint']}</param>
+                </state_interface>
+            </joint>
+        </ros2_control>
         <!-- <gazebo>
             <plugin filename="libign_ros2_control-system.so"

File: software/ros_packages/rover_urdf/urdf/rover2_body.urdf.xacro (robot description, xacro)
@@ -4,5 +4,10 @@
 -->
 <robot name="rover_body" xmlns:xacro="https://ros.org/wiki/xacro">
-    <xacro:macro name="rover_body" params="name:=rover">
+    <xacro:macro name="rover_body" params="name:=rover hardware_type:=main">
+        <!-- Set wheel direction -->
+        <xacro:property name="wheel_direction" value="1.0"/>
+        <xacro:if value="${hardware_type == 'main'}">
+            <xacro:property name="wheel_direction" value="-1.0"/>
+        </xacro:if>
         <!-- Main Body -->
         <link name="${name}_base_origin">
@@ -435,5 +440,5 @@
             <parent link="${name}_right_bogie"/>
             <child link="${name}_front_right_wheel"/>
-            <axis xyz="1.0 -0.0 0.0"/>
+            <axis xyz="${wheel_direction} 0.0 0.0"/>
         </joint>
         <joint name="${name}_middle_right_wheel_joint" type="continuous">
@@ -441,5 +446,5 @@
             <parent link="${name}_right_bogie"/>
             <child link="${name}_middle_right_wheel"/>
-            <axis xyz="1.0 0.0 0.0"/>
+            <axis xyz="${wheel_direction} 0.0 0.0"/>
         </joint>
         <joint name="${name}_back_right_wheel_joint" type="continuous">
@@ -447,5 +452,5 @@
             <parent link="${name}_rear_bogie"/>
             <child link="${name}_back_right_wheel"/>
-            <axis xyz="1.0 0.0 0.0"/>
+            <axis xyz="${wheel_direction} 0.0 0.0"/>
         </joint>
         <gazebo reference="${name}_base_origin">
@@ -476,5 +481,5 @@
             <sensor name="gps" type="navsat">
                 <always_on>true</always_on>
-                <update_rate>100</update_rate>
+                <update_rate>5</update_rate>
                 <visualize>true</visualize>
                 <topic>gps/raw</topic>
@@ -489,5 +494,5 @@
                             <noise type="gaussian">
                                 <mean>0.0</mean>
-                                <stddev>1.5e-5</stddev>   <!-- meters -->
+                                <stddev>1.5e-6</stddev>   <!-- meters -->
                             </noise>
                         </horizontal>
@@ -495,5 +500,5 @@
                             <noise type="gaussian">
                                 <mean>0.0</mean>
-                                <stddev>3.0</stddev>
+                                <stddev>1.0</stddev>
                             </noise>
                         </vertical>

File: software/ros_packages/rover_urdf/urdf/rover2_urdf.xacro (robot description, xacro)
@@ -4,5 +4,5 @@
 -->
 <robot name="rover" xmlns:xacro="https://ros.org/wiki/xacro">
-    <xacro:macro name="rover" params="name attachment:=arm">
+    <xacro:macro name="rover" params="name attachment:=arm hardware_type:=main">
         <!-- Includes (material libraries, etc) -->
         <xacro:include filename="$(find rover_arm_urdf)/urdf/rover2_arm.urdf.xacro" />
@@ -10,5 +10,5 @@
         <xacro:include filename="$(find rover_urdf)/urdf/materials.xacro" />
         <!-- Link Chasis with bogies and tower -->
-        <xacro:rover_body name="rover">
+        <xacro:rover_body name="rover" hardware_type="${hardware_type}">
         </xacro:rover_body>
         <!-- Link Arm or Scimech-->
