Commit message: Configured planners and moveit to run. Still need servo.

File: software/ros_packages/rover2_arm/config/rover.ros2_control.xacro (robot description, xacro)
@@ -1,12 +1,19 @@
 <?xml version="1.0"?>
 <robot xmlns:xacro="http://www.ros.org/wiki/xacro">
-    <xacro:macro name="rover_ros2_control" params="name initial_positions_file">
+    <xacro:macro name="rover_ros2_control" params="name initial_positions_file ros2_control_hardware_type:=main">
         <xacro:property name="initial_positions" value="${load_yaml(initial_positions_file)['initial_positions']}"/>
         <ros2_control name="${name}" type="system">
             <hardware>
-                <!-- By default, set up controllers for simulation. This won't work on real hardware -->
+              <xacro:if value="${ros2_control_hardware_type == 'main'}">
+                <plugin>odrive_ros2_control_plugin/ODriveHardwareInterface</plugin>
+                <param name="can">can1</param>
+              </xacro:if>
+              <xacro:if value="${ros2_control_hardware_type == 'sim'}">
                 <plugin>mock_components/GenericSystem</plugin>
+              </xacro:if>
             </hardware>
             <joint name="rover_arm_base_joint">
+                <param name="node_id">0</param>
+                <param name="gear_ratio">400.0</param>
                 <command_interface name="position"/>
                 <command_interface name="velocity"/>
@@ -17,4 +24,6 @@
             </joint>
             <joint name="rover_arm_shoulder_joint">
+                <param name="node_id">1</param>
+                <param name="gear_ratio">640.0</param>
                 <command_interface name="position"/>
                 <command_interface name="velocity"/>
@@ -25,4 +34,6 @@
             </joint>
             <joint name="rover_arm_elbow_pitch_joint">
+                <param name="node_id">2</param>
+                <param name="gear_ratio">393.6</param>
                 <command_interface name="position"/>
                 <command_interface name="velocity"/>
@@ -33,4 +44,6 @@
             </joint>
             <joint name="rover_arm_elbow_roll_joint">
+                <param name="node_id">3</param>
+                <param name="gear_ratio">120.0</param>
                 <command_interface name="position"/>
                 <command_interface name="velocity"/>
@@ -41,4 +54,6 @@
             </joint>
             <joint name="rover_arm_wrist_pitch_joint">
+                <param name="node_id">4</param>
+                <param name="gear_ratio">370.0</param>
                 <command_interface name="position"/>
                 <command_interface name="velocity"/>
@@ -49,4 +64,6 @@
             </joint>
             <joint name="rover_arm_wrist_roll_joint">
+                <param name="node_id">5</param>
+                <param name="gear_ratio">100.0</param>
                 <command_interface name="position"/>
                 <command_interface name="velocity"/>

File: software/ros_packages/rover2_arm/config/rover.urdf.xacro (robot description, xacro)
@@ -2,8 +2,15 @@
 <robot xmlns:xacro="http://www.ros.org/wiki/xacro" name="rover">
     <xacro:arg name="initial_positions_file" default="initial_positions.yaml" />
+    <xacro:arg name="ros2_control_hardware_type" default="main" />
     <!-- Import rover urdf file -->
     <xacro:include filename="$(find rover_urdf)/urdf/rover_urdf.xacro" />
     <!-- Import control_xacro -->
     <xacro:include filename="rover.ros2_control.xacro" />
-    <xacro:rover_ros2_control name="FakeSystem" initial_positions_file="$(arg initial_positions_file)"/>
+    <!-- Include sensors and other links -->
+    <xacro:include filename="$(find realsense2_description)/urdf/_d405.urdf.xacro"/>
+    <!-- Instantiate micros  -->
+    <xacro:sensor_d405 parent ="rover_arm_gripper" name="d405" use_nominal_extrinsics="true">
+        <origin xyz="0 0.04075 0.1" rpy="0 -1.3963 -1.5708"/>
+    </xacro:sensor_d405>
+    <xacro:rover_ros2_control name="FakeSystem" initial_positions_file="$(arg initial_positions_file)" ros2_control_hardware_type="$(arg ros2_control_hardware_type)"/>
 </robot>

Commit message: New Arm Package Working

File: software/ros_packages/rover2_arm/config/rover.ros2_control.xacro (robot description, xacro)
@@ -7,5 +7,5 @@
               <xacro:if value="${ros2_control_hardware_type == 'main'}">
                 <plugin>odrive_ros2_control_plugin/ODriveHardwareInterface</plugin>
-                <param name="can">can1</param>
+                <param name="can">can0</param>
               </xacro:if>
               <xacro:if value="${ros2_control_hardware_type == 'sim'}">

File: software/ros_packages/rover2_arm/config/rover.urdf.xacro (robot description, xacro)
@@ -11,5 +11,6 @@
     <!-- Instantiate micros  -->
     <xacro:sensor_d405 parent ="rover_arm_gripper" name="d405" use_nominal_extrinsics="true">
-        <origin xyz="0 0.04075 0.1" rpy="0 -1.3963 -1.5708"/>
+        <!-- For older urdf <origin xyz="0 0.04075 0.1" rpy="0 -1.3963 -1.5708"/> -->
+        <origin xyz="-0.001611 -0.040711 0.099525" rpy="0.0 -1.3963635 1.5707963"/>
     </xacro:sensor_d405>
     <xacro:rover_ros2_control name="FakeSystem" initial_positions_file="$(arg initial_positions_file)" ros2_control_hardware_type="$(arg ros2_control_hardware_type)"/>

File: software/ros_packages/rover_urdf/urdf/rover_urdf.xacro (robot description, xacro)
@@ -6,5 +6,5 @@
     <xacro:macro name="rover" params="name attachment:=arm">
         <!-- Includes (material libraries, etc) -->
-        <xacro:include filename="$(find rover_arm_urdf)/urdf/rover_arm.urdf.xacro" />
+        <xacro:include filename="$(find rover_arm_urdf)/urdf/rover2_arm.urdf.xacro" />
         <xacro:include filename="rover_body.urdf.xacro"/>
         <!-- Link Chasis with bogies and tower -->
@@ -13,7 +13,7 @@
         <!-- Link Arm or Scimech-->
         <xacro:if value="${attachment== 'arm'}">
-            <xacro:rover_arm parent="rover_base_origin" >
+            <xacro:rover2_arm parent="rover_base_origin" >
                 <origin rpy= "0.0 0.0 0.0" xyz="0.175735 0 0.03175"/>
-            </xacro:rover_arm>
+            </xacro:rover2_arm>
         </xacro:if>
         <xacro:if value="${attachment == 'science'}">

Commit message: Moved firmware in software to electrical, fixed script-dir, and created gazebo for DT

File: software/ros_packages/rover2_arm/config/rover.ros2_control.xacro (robot description, xacro)
@@ -2,5 +2,5 @@
 <robot xmlns:xacro="http://www.ros.org/wiki/xacro">
     <xacro:macro name="rover_ros2_control" params="name initial_positions_file ros2_control_hardware_type:=main">
-        <xacro:property name="initial_positions" value="${load_yaml(initial_positions_file)['initial_positions']}"/>
+        <xacro:property name="initial_positions" value="${xacro.load_yaml(initial_positions_file)['initial_positions']}"/>
         <ros2_control name="${name}" type="system">
             <hardware>
@@ -11,4 +11,7 @@
               <xacro:if value="${ros2_control_hardware_type == 'sim'}">
                 <plugin>mock_components/GenericSystem</plugin>
+              </xacro:if>
+              <xacro:if value="${ros2_control_hardware_type == 'gazebo'}">
+                <plugin>fake_components/GenericSystem</plugin>
               </xacro:if>
             </hardware>

File: software/ros_packages/rover2_arm/config/rover.urdf.xacro (robot description, xacro)
@@ -4,6 +4,9 @@
     <xacro:arg name="ros2_control_hardware_type" default="main" />
     <xacro:arg name="drive_initial_positions_file" default="$(find rover_urdf)/ros2_control/initial_positions.yaml" />
+    <xacro:arg name="attachment" default="arm" />
+    <xacro:property name="hardware_type" value="$(arg ros2_control_hardware_type)"/>
     <!-- Import rover urdf file -->
     <xacro:include filename="$(find rover_urdf)/urdf/rover2_urdf.xacro" />
+    <xacro:rover name="rover" attachment="$(arg attachment)"/>
     <!-- Import control_xacro -->
     <xacro:include filename="rover.ros2_control.xacro" />
@@ -12,11 +15,13 @@
     <xacro:include filename="$(find realsense2_description)/urdf/_d405.urdf.xacro"/>
     <!-- Instantiate micros  -->
-    <xacro:sensor_d405 parent ="rover_arm_gripper" name="d405" use_nominal_extrinsics="true">
-        <!-- For older urdf <origin xyz="0 0.04075 0.1" rpy="0 -1.3963 -1.5708"/> -->
-        <origin xyz="-0.001611 -0.040711 0.099525" rpy="0.0 -1.3963635 1.5707963"/>
-    </xacro:sensor_d405>
+    <xacro:unless value="${hardware_type == 'gazebo'}">
+        <xacro:sensor_d405 parent ="rover_arm_gripper" name="d405" use_nominal_extrinsics="true">
+            <!-- For older urdf <origin xyz="0 0.04075 0.1" rpy="0 -1.3963 -1.5708"/> -->
+            <origin xyz="-0.001611 -0.040711 0.099525" rpy="0.0 -1.3963635 1.5707963"/>
+        </xacro:sensor_d405>
     <!-- Include rover arm ros2_control -->
-    <xacro:rover_ros2_control name="rover_arm" initial_positions_file="$(arg initial_positions_file)" ros2_control_hardware_type="$(arg ros2_control_hardware_type)"/>
+        <xacro:rover_ros2_control name="rover_arm" initial_positions_file="$(arg initial_positions_file)" ros2_control_hardware_type="$(arg ros2_control_hardware_type)"/>
+    </xacro:unless>
     <!-- Include rover drive ros2_control -->
-    <xacro:rover_body_ros2_control name="rover_drive" initial_positions_file="$(arg drive_initial_positions_file)" ros2_control_hardware_type="sim"/>
+    <xacro:rover_body_ros2_control name="rover_drive" initial_positions_file="$(arg drive_initial_positions_file)" ros2_control_hardware_type="gazebo"/>
 </robot>

File: software/ros_packages/rover_urdf/ros2_control/rover_body.ros2_control.xacro (robot description, xacro)
@@ -2,14 +2,17 @@
 <robot xmlns:xacro="http://www.ros.org/wiki/xacro">
     <xacro:macro name="rover_body_ros2_control" params="name initial_positions_file ros2_control_hardware_type:=main">
-        <xacro:property name="initial_positions" value="${load_yaml(initial_positions_file)['initial_positions']}"/>
+        <xacro:property name="initial_positions" value="${xacro.load_yaml(initial_positions_file)['initial_positions']}"/>
         <ros2_control name="${name}" type="system">
             <hardware>
-              <xacro:if value="${ros2_control_hardware_type == 'main'}">
-                <plugin>odrive_ros2_control_plugin/ODriveHardwareInterface</plugin>
-                <param name="can">can0</param>
-              </xacro:if>
-              <xacro:if value="${ros2_control_hardware_type == 'sim'}">
-                <plugin>mock_components/GenericSystem</plugin>
-              </xacro:if>
+                <xacro:if value="${ros2_control_hardware_type == 'main'}">
+                    <plugin>odrive_ros2_control_plugin/ODriveHardwareInterface</plugin>
+                    <param name="can">can0</param>
+                </xacro:if>
+                <xacro:if value="${ros2_control_hardware_type == 'sim'}">
+                    <plugin>mock_components/GenericSystem</plugin>
+                </xacro:if>
+                <xacro:if value="${ros2_control_hardware_type == 'gazebo'}">
+                    <plugin>fake_components/GenericSystem</plugin>
+                </xacro:if>
             </hardware>
             <joint name="rover_front_left_link_joint">

File: software/ros_packages/rover_urdf/urdf/rover2_urdf.xacro (robot description, xacro)
@@ -22,4 +22,3 @@
             <!-- Arm option for gripper -->
     </xacro:macro>
-    <xacro:rover name="rover" attachment="arm"/>
 </robot>
