Commit message: Rover Gazebo package with sensor and worlds

File: software/ros_packages/rover2_arm/config/rover.ros2_control.xacro (robot description, xacro)
@@ -13,5 +13,5 @@
               </xacro:if>
               <xacro:if value="${ros2_control_hardware_type == 'gazebo'}">
-                <plugin>fake_components/GenericSystem</plugin>
+                <plugin>ign_ros2_control/GazeboSystem</plugin>
               </xacro:if>
             </hardware>

File: software/ros_packages/rover2_arm/config/rover.urdf.xacro (robot description, xacro)
@@ -6,4 +6,5 @@
     <xacro:arg name="attachment" default="arm" />
     <xacro:property name="hardware_type" value="$(arg ros2_control_hardware_type)"/>
+    <xacro:property name="front_attachment" value = "$(arg attachment)"/>
     <!-- Import rover urdf file -->
     <xacro:include filename="$(find rover_urdf)/urdf/rover2_urdf.xacro" />
@@ -12,16 +13,9 @@
     <xacro:include filename="rover.ros2_control.xacro" />
     <xacro:include filename="$(find rover_urdf)/ros2_control/rover_body.ros2_control.xacro" />
-    <!-- Include sensors and other links -->
-    <xacro:include filename="$(find realsense2_description)/urdf/_d405.urdf.xacro"/>
-    <!-- Instantiate micros  -->
-    <xacro:unless value="${hardware_type == 'gazebo'}">
-        <xacro:sensor_d405 parent ="rover_arm_gripper" name="d405" use_nominal_extrinsics="true">
-            <!-- For older urdf <origin xyz="0 0.04075 0.1" rpy="0 -1.3963 -1.5708"/> -->
-            <origin xyz="-0.001611 -0.040711 0.099525" rpy="0.0 -1.3963635 1.5707963"/>
-        </xacro:sensor_d405>
     <!-- Include rover arm ros2_control -->
+    <xacro:if value="${front_attachment == 'arm'}">
         <xacro:rover_ros2_control name="rover_arm" initial_positions_file="$(arg initial_positions_file)" ros2_control_hardware_type="$(arg ros2_control_hardware_type)"/>
-    </xacro:unless>
+    </xacro:if>
     <!-- Include rover drive ros2_control -->
-    <xacro:rover_body_ros2_control name="rover_drive" initial_positions_file="$(arg drive_initial_positions_file)" ros2_control_hardware_type="gazebo"/>
+    <xacro:rover_body_ros2_control name="rover_drive" initial_positions_file="$(arg drive_initial_positions_file)" ros2_control_hardware_type="$(arg ros2_control_hardware_type)"/>
 </robot>

File: software/ros_packages/rover_urdf/ros2_control/rover_body.ros2_control.xacro (robot description, xacro)
@@ -6,6 +6,7 @@
             <hardware>
                 <xacro:if value="${ros2_control_hardware_type == 'main'}">
-                    <plugin>odrive_ros2_control_plugin/ODriveHardwareInterface</plugin>
-                    <param name="can">can0</param>
+                    <!-- <plugin>odrive_ros2_control_plugin/ODriveHardwareInterface</plugin>
+                    <param name="can">can0</param> -->
+                    <plugin>mock_components/GenericSystem</plugin>
                 </xacro:if>
                 <xacro:if value="${ros2_control_hardware_type == 'sim'}">
@@ -13,5 +14,5 @@
                 </xacro:if>
                 <xacro:if value="${ros2_control_hardware_type == 'gazebo'}">
-                    <plugin>fake_components/GenericSystem</plugin>
+                    <plugin>gz_ros2_control/GazeboSimSystem</plugin>
                 </xacro:if>
             </hardware>
@@ -66,5 +67,5 @@
                 <param name="node_id">0</param>
                 <param name="gear_ratio">50</param>
-                <command_interface name="position"/>
+                <!-- <command_interface name="position"/> -->
                 <command_interface name="velocity"/>
                 <state_interface name="position">
@@ -76,5 +77,5 @@
                 <param name="node_id">2</param>
                 <param name="gear_ratio">50</param>
-                <command_interface name="position"/>
+                <!-- <command_interface name="position"/> -->
                 <command_interface name="velocity"/>
                 <state_interface name="position">
@@ -86,5 +87,5 @@
                 <param name="node_id">4</param>
                 <param name="gear_ratio">50</param>
-                <command_interface name="position"/>
+                <!-- <command_interface name="position"/> -->
                 <command_interface name="velocity"/>
                 <state_interface name="position">
@@ -96,5 +97,5 @@
                 <param name="node_id">1</param>
                 <param name="gear_ratio">50</param>
-                <command_interface name="position"/>
+                <!-- <command_interface name="position"/> -->
                 <command_interface name="velocity"/>
                 <state_interface name="position">
@@ -106,5 +107,5 @@
                 <param name="node_id">3</param>
                 <param name="gear_ratio">50</param>
-                <command_interface name="position"/>
+                <!-- <command_interface name="position"/> -->
                 <command_interface name="velocity"/>
                 <state_interface name="position">
@@ -116,5 +117,5 @@
                 <param name="node_id">5</param>
                 <param name="gear_ratio">50</param>
-                <command_interface name="position"/>
+                <!-- <command_interface name="position"/> -->
                 <command_interface name="velocity"/>
                 <state_interface name="position">
@@ -124,4 +125,14 @@
             </joint>
         </ros2_control>
+        <!-- <gazebo>
+            <plugin filename="libign_ros2_control-system.so"
+                    name="ign_ros2_control::System">
+            </plugin>
+        </gazebo> -->
+        <gazebo>
+            <plugin filename="libgz_ros2_control-system.so" name="gz_ros2_control::GazeboSimROS2ControlPlugin">
+                <parameters>$(find rover2_control)/config/rover_drive.yaml</parameters>
+            </plugin>
+        </gazebo>
     </xacro:macro>
 </robot>

File: software/ros_packages/rover_urdf/urdf/rover2_body.urdf.xacro (robot description, xacro)
@@ -349,6 +349,7 @@
             <axis xyz="0.0 1.0 0.0"/>
             <limit upper="0.2617994" lower="-0.2617994" effort="100" velocity="100"/>
-        </joint>
-        <joint name="${name}_front_left_link_joint" type="revolute">
+            <dynamics damping="2.0" friction="0.2"/>
+        </joint>
+        <joint name="${name}_front_left_link_joint" type="fixed">
             <origin xyz="0.244132 0.178623 0.051277" rpy="0 0 1.5708"/>
             <parent link="${name}_base_origin"/>
@@ -356,13 +357,14 @@
             <axis xyz="1.0 0.0 0.0"/>
             <limit upper="0.2617994" lower="-0.2617994" effort="100" velocity="100"/>
-        </joint>
-        <joint name="${name}_back_left_link_joint" type="revolute">
+            <dynamics damping="2.0" friction="0.2"/>
+        </joint>
+        <joint name="${name}_back_left_link_joint" type="fixed">
             <origin xyz="0.170002 0.178623 0.051277" rpy="0 0 1.5708"/>
             <parent link="${name}_base_origin"/>
             <child link="${name}_back_left_link"/>
-            <axis xyz="1.0 0.0 0.0"/>
-            <limit upper="0.2617994" lower="-0.2617994" effort="100" velocity="100"/>
-        </joint>
-        <joint name="${name}_front_left_bogie_joint" type="continuous">
+            <!-- <axis xyz="1.0 0.0 0.0"/>
+            <limit upper="0.2617994" lower="-0.2617994" effort="100" velocity="100"/> -->
+        </joint>
+        <joint name="${name}_front_left_bogie_joint" type="fixed">
             <origin xyz="0.036626 0.062229 -0.077732" rpy="0 0 0"/>
             <parent link="${name}_front_left_link"/>
@@ -370,4 +372,5 @@
             <axis xyz="1.0 0.0 -0.0"/>
             <limit upper="0.2617994" lower="-0.2617994" effort="100" velocity="100"/>
+            <dynamics damping="2.0" friction="0.2"/>
         </joint>
         <!-- Four Bars Don't exist in URDF's See mimic for Parallel four bars -->
@@ -379,5 +382,5 @@
             <limit upper="0.2617994" lower="-0.2617994" effort="100" velocity="100"/>
         </joint> -->
-        <joint name="${name}_front_right_link_joint" type="revolute">
+        <joint name="${name}_front_right_link_joint" type="fixed">
             <origin xyz="0.244132 -0.220157 0.051277" rpy="0 0 1.5708"/>
             <parent link="${name}_base_origin"/>
@@ -385,16 +388,19 @@
             <axis xyz="1.0 0.0 0.0"/>
             <limit upper="0.2617994" lower="-0.2617994" effort="100" velocity="100"/>
-        </joint>
-        <joint name="${name}_back_right_link_joint" type="continuous">
+            <dynamics damping="2.0" friction="0.2"/>
+        </joint>
+        <joint name="${name}_back_right_link_joint" type="fixed">
             <origin xyz="0.170002 -0.220157 0.051277" rpy="0 0 1.5708"/>
             <parent link="${name}_base_origin"/>
             <child link="${name}_back_right_link"/>
-            <axis xyz="1.0 0.0 0.0"/>
-        </joint>
-        <joint name="${name}_front_right_bogie_joint" type="continuous">
+            <!-- <axis xyz="1.0 0.0 0.0"/> -->
+        </joint>
+        <joint name="${name}_front_right_bogie_joint" type="fixed">
             <origin xyz="-0.036626 0.054471 -0.076141" rpy="0 0 0"/>
             <parent link="${name}_front_right_link"/>
             <child link="${name}_right_bogie"/>
             <axis xyz="-1.0 0.0 0.0"/>
+            <limit upper="0.2617994" lower="-0.2617994" effort="100" velocity="100"/>
+            <dynamics damping="2.0" friction="0.2"/>
         </joint>
         <!-- Four bars don't exist in URDF's -->
@@ -411,5 +417,5 @@
             <parent link="${name}_left_bogie"/>
             <child link="${name}_front_left_wheel"/>
-            <axis xyz="-1.0 0.0 0.0"/>
+            <axis xyz="1.0 0.0 0.0"/>
         </joint>
         <joint name="${name}_back_left_wheel_joint" type="continuous">
@@ -423,5 +429,5 @@
             <parent link="${name}_left_bogie"/>
             <child link="${name}_middle_left_wheel"/>
-            <axis xyz="-1.0 0.0 0.0"/>
+            <axis xyz="1.0 0.0 0.0"/>
         </joint>
         <joint name="${name}_front_right_wheel_joint" type="continuous">
@@ -429,5 +435,5 @@
             <parent link="${name}_right_bogie"/>
             <child link="${name}_front_right_wheel"/>
-            <axis xyz="-1.0 -0.0 0.0"/>
+            <axis xyz="1.0 -0.0 0.0"/>
         </joint>
         <joint name="${name}_middle_right_wheel_joint" type="continuous">
@@ -435,5 +441,5 @@
             <parent link="${name}_right_bogie"/>
             <child link="${name}_middle_right_wheel"/>
-            <axis xyz="-1.0 0.0 0.0"/>
+            <axis xyz="1.0 0.0 0.0"/>
         </joint>
         <joint name="${name}_back_right_wheel_joint" type="continuous">
@@ -443,4 +449,57 @@
             <axis xyz="1.0 0.0 0.0"/>
         </joint>
+        <gazebo reference="${name}_base_origin">
+            <sensor name="imu_sensor" type="imu">
+                <always_on>1</always_on>
+                <update_rate>100</update_rate>
+                <visualize>true</visualize>
+                <topic>imu/data/raw</topic>
+                <ignition_frame_id>${name}_base_origin</ignition_frame_id>
+                <plugin filename="gz-sim-imu-system"
+                    name="gz::sim::systems::Imu">
+                </plugin>
+            </sensor>
+        </gazebo>
+        <gazebo reference="${name}_base_origin">
+            <sensor name="imu_mag" type="magnetometer">
+                <always_on>1</always_on>
+                <update_rate>100</update_rate>
+                <visualize>true</visualize>
+                <topic>imu/mag/raw</topic>
+                <ignition_frame_id>${name}_base_origin</ignition_frame_id>
+                <plugin filename="ignition-gazebo-magnetometer-system"
+                    name="ignition::gazebo::systems::Magnetometer">
+                </plugin>
+            </sensor>
+        </gazebo>
+        <gazebo reference="${name}_base_origin">
+            <sensor name="gps" type="navsat">
+                <always_on>true</always_on>
+                <update_rate>100</update_rate>
+                <visualize>true</visualize>
+                <topic>gps/raw</topic>
+                <ignition_frame_id>${name}_base_origin</ignition_frame_id>
+                <plugin
+                    filename="ignition-gazebo-navsat-system"
+                    name="ignition::gazebo::systems::NavSat">
+                </plugin>
+                <navsat>
+                    <position_sensing>
+                        <horizontal>
+                            <noise type="gaussian">
+                                <mean>0.0</mean>
+                                <stddev>1.5e-5</stddev>   <!-- meters -->
+                            </noise>
+                        </horizontal>
+                        <vertical>
+                            <noise type="gaussian">
+                                <mean>0.0</mean>
+                                <stddev>3.0</stddev>
+                            </noise>
+                        </vertical>
+                    </position_sensing>
+                </navsat>
+            </sensor>
+        </gazebo>
     </xacro:macro>
 </robot>

File: software/ros_packages/rover_urdf/urdf/rover2_urdf.xacro (robot description, xacro)
@@ -17,8 +17,71 @@
                 <origin rpy= "0.0 0.0 0.0" xyz="0.173803 -0.020767 0.071924"/>
             </xacro:rover2_arm>
+            <!-- Include sensors and other links -->
+            <xacro:include filename="$(find realsense2_description)/urdf/_d405.urdf.xacro"/>
+            <!-- Instantiate micros  -->
+            <xacro:sensor_d405 parent ="rover_arm_gripper" name="d405" use_nominal_extrinsics="true">
+                <!-- For older urdf <origin xyz="0 0.04075 0.1" rpy="0 -1.3963 -1.5708"/> -->
+                <origin xyz="-0.001611 -0.040711 0.099525" rpy="0.0 -1.3963635 1.5707963"/>
+            </xacro:sensor_d405>
         </xacro:if>
         <xacro:if value="${attachment == 'science'}">
         </xacro:if>
+        <!-- Sensors -->
+        <!-- Chassis Depth Camera -->
+        <xacro:include filename="$(find realsense2_description)/urdf/_d455.urdf.xacro"/>
+        <xacro:sensor_d455 parent="rover_base_origin" name="d455" use_nominal_extrinsics="true">
+            <origin xyz="0.26 0.11 0.15" rpy="3.1415926536 0.2618 0"/>
+        </xacro:sensor_d455>
             <!-- Arm option for gripper -->
+        <!-- Gazebo Setup -->
+        <gazebo reference="d455_depth_frame">
+            <sensor name="d455" type="rgbd_camera">
+                <ignition_frame_id>d455_depth_frame</ignition_frame_id>
+                <camera name="d455">
+                <horizontal_fov>1.518436</horizontal_fov>
+                <!-- <lens> Camera Specific (Don't know them)
+                    <intrinsics>
+                    <fx>277.1</fx>
+                    <fy>277.1</fy>
+                    <cx>160.5</cx>
+                    <cy>120.5</cy>
+                    <s>0</s>
+                    </intrinsics>
+                </lens>
+                <distortion>
+                    <k1>0.104207</k1>
+                    <k2>-0.255558</k2>
+                    <k3>0.128694</k3>
+                    <p1>0.000512</p1>
+                    <p2>0.000319</p2>
+                    <center>0.5 0.5</center>
+                </distortion> -->
+                <image>
+                    <width>1280</width>
+                    <height>720</height>
+                    <format>R_FLOAT32</format>
+                </image>
+                <clip>
+                    <near>0.1</near>
+                    <far>10</far>
+                </clip>
+                <depth_camera>
+                    <clip>
+                    <near>0.6</near>
+                    <far>6</far>
+                    </clip>
+                </depth_camera>
+                <noise>
+                    <type>gaussian</type>
+                    <mean>0</mean>
+                    <stddev>0.01</stddev>
+                </noise>
+                </camera>
+                <always_on>1</always_on>
+                <update_rate>15</update_rate>
+                <visualize>true</visualize>
+                <topic>/camera/d455/depth/color</topic>
+            </sensor>
+        </gazebo>
     </xacro:macro>
 </robot>

Commit message: funky yaml

File: software/ros_packages/rover2_arm/config/rover.ros2_control.xacro (robot description, xacro)
@@ -7,5 +7,5 @@
               <xacro:if value="${ros2_control_hardware_type == 'main'}">
                 <plugin>odrive_ros2_control_plugin/ODriveHardwareInterface</plugin>
-                <param name="can">can0</param>
+                <param name="can">can1</param>
               </xacro:if>
               <xacro:if value="${ros2_control_hardware_type == 'sim'}">

File: software/ros_packages/rover_arm/config/rover_arm.urdf.xacro (robot description, xacro)
@@ -3,6 +3,12 @@
     <xacro:arg name="initial_positions_file" default="initial_positions.yaml" />
     <xacro:arg name="ros2_control_hardware_type" default="main" />
+    <xacro:include filename="$(find rover_urdf)/urdf/rover_body.urdf.xacro" />
+    <xacro:rover_body name="rover_body">
+    </xacro:rover_body>
     <!-- Import rover_arm urdf file -->
     <xacro:include filename="$(find rover_arm_urdf)/urdf/rover_arm.urdf" />
+    <xacro:rover_arm parent="rover_base_origin">
+        <origin xyz="0 0 0" rpy="0 0 0"/>
+    </xacro:sensor_d455>
     <!-- Import control_xacro -->
     <xacro:include filename="rover_arm.ros2_control.xacro" />

File: software/ros_packages/rover_urdf/ros2_control/rover_body.ros2_control.xacro (robot description, xacro)
@@ -6,6 +6,6 @@
             <hardware>
                 <xacro:if value="${ros2_control_hardware_type == 'main'}">
-                    <!-- <plugin>odrive_ros2_control_plugin/ODriveHardwareInterface</plugin>
-                    <param name="can">can0</param> -->
+                    <plugin>odrive_ros2_control_plugin/ODriveHardwareInterface</plugin>
+                    <param name="can">can0</param>
                     <plugin>mock_components/GenericSystem</plugin>
                 </xacro:if>
@@ -17,5 +17,5 @@
                 </xacro:if>
             </hardware>
-            <joint name="rover_front_left_link_joint">
+            <!-- <joint name="rover_front_left_link_joint">
                 <state_interface name="position">
                     <param name="initial_value">${initial_positions['rover_front_left_link_joint']}</param>
@@ -31,5 +31,5 @@
                     <param name="initial_value">${initial_positions['rover_front_left_bogie_joint']}</param>
                 </state_interface>
-            </joint>
+            </joint> -->
             <!-- Four Bar linkage doesn't exist in URDF's -->
             <!-- <joint name="rover_back_left_bogie_joint">
@@ -38,5 +38,5 @@
                 </state_interface>
             </joint> -->
-            <joint name="rover_front_right_link_joint">
+            <!--<joint name="rover_front_right_link_joint">
                 <state_interface name="position">
                     <param name="initial_value">${initial_positions['rover_front_right_link_joint']}</param>
@@ -52,5 +52,5 @@
                     <param name="initial_value">${initial_positions['rover_front_right_bogie_joint']}</param>
                 </state_interface>
-            </joint>
+            </joint>-->
             <!-- Four Bar linkage doesn't exist in URDF's -->
             <!-- <joint name="rover_back_right_bogie_joint">
@@ -59,9 +59,9 @@
                 </state_interface>
             </joint> -->
-            <joint name="rover_rear_bogie_joint">
+            <!--<joint name="rover_rear_bogie_joint">
                 <state_interface name="position">
                     <param name="initial_value">${initial_positions['rover_rear_bogie_joint']}</param>
                 </state_interface>
-            </joint>
+            </joint>-->
             <joint name="rover_front_left_wheel_joint">
                 <param name="node_id">0</param>

File: software/ros_packages/rover_urdf/urdf/rover2_body.urdf.xacro (robot description, xacro)
@@ -435,5 +435,5 @@
             <parent link="${name}_right_bogie"/>
             <child link="${name}_front_right_wheel"/>
-            <axis xyz="1.0 -0.0 0.0"/>
+            <axis xyz="-1.0 -0.0 0.0"/>
         </joint>
         <joint name="${name}_middle_right_wheel_joint" type="continuous">
@@ -441,5 +441,5 @@
             <parent link="${name}_right_bogie"/>
             <child link="${name}_middle_right_wheel"/>
-            <axis xyz="1.0 0.0 0.0"/>
+            <axis xyz="-1.0 0.0 0.0"/>
         </joint>
         <joint name="${name}_back_right_wheel_joint" type="continuous">
@@ -447,5 +447,5 @@
             <parent link="${name}_rear_bogie"/>
             <child link="${name}_back_right_wheel"/>
-            <axis xyz="1.0 0.0 0.0"/>
+            <axis xyz="-1.0 0.0 0.0"/>
         </joint>
         <gazebo reference="${name}_base_origin">
