Commit message: move perp to plane, Northrop arm, small bugs

File: software/ros_packages/rover2_arm/config/rover.ros2_control.xacro (robot description, xacro)
@@ -1,5 +1,5 @@
 <?xml version="1.0"?>
 <robot xmlns:xacro="http://www.ros.org/wiki/xacro">
-    <xacro:macro name="rover_ros2_control" params="name initial_positions_file ros2_control_hardware_type:=main">
+    <xacro:macro name="rover_ros2_control" params="name initial_positions_file ros2_control_hardware_type:=main attachment:=arm">
         <xacro:property name="initial_positions" value="${xacro.load_yaml(initial_positions_file)['initial_positions']}"/>
         <ros2_control name="${name}" type="system">
@@ -18,5 +18,10 @@
             <joint name="rover_arm_base_joint">
                 <param name="node_id">0</param>
-                <param name="gear_ratio">400.0</param>
+                <xacro:if value="${attachment == 'arm'}">
+                  <param name="gear_ratio">400.0</param>
+                </xacro:if>
+                <xacro:if value="${attachment == 'northrop_arm'}">
+                  <param name="gear_ratio">1.0</param>
+                </xacro:if>
                 <command_interface name="position"/>
                 <command_interface name="velocity"/>
@@ -28,5 +33,10 @@
             <joint name="rover_arm_shoulder_joint">
                 <param name="node_id">1</param>
-                <param name="gear_ratio">640.0</param>
+                <xacro:if value="${attachment == 'arm'}">
+                  <param name="gear_ratio">640.0</param>
+                </xacro:if>
+                <xacro:if value="${attachment == 'northrop_arm'}">
+                  <param name="gear_ratio">1.0</param>
+                </xacro:if>
                 <command_interface name="position"/>
                 <command_interface name="velocity"/>
@@ -38,5 +48,10 @@
             <joint name="rover_arm_elbow_pitch_joint">
                 <param name="node_id">2</param>
-                <param name="gear_ratio">393.6</param>
+                <xacro:if value="${attachment == 'arm'}">
+                  <param name="gear_ratio">393.6</param>
+                </xacro:if>
+                <xacro:if value="${attachment == 'northrop_arm'}">
+                  <param name="gear_ratio">1.0</param>
+                </xacro:if>
                 <command_interface name="position"/>
                 <command_interface name="velocity"/>
@@ -48,5 +63,10 @@
             <joint name="rover_arm_elbow_roll_joint">
                 <param name="node_id">3</param>
-                <param name="gear_ratio">120.0</param>
+                <xacro:if value="${attachment == 'arm'}">
+                  <param name="gear_ratio">120.0</param>
+                </xacro:if>
+                <xacro:if value="${attachment == 'northrop_arm'}">
+                  <param name="gear_ratio">1.0</param>
+                </xacro:if>
                 <command_interface name="position"/>
                 <command_interface name="velocity"/>
@@ -58,5 +78,10 @@
             <joint name="rover_arm_wrist_pitch_joint">
                 <param name="node_id">4</param>
-                <param name="gear_ratio">370.0</param>
+                <xacro:if value="${attachment == 'arm'}">
+                  <param name="gear_ratio">370.0</param>
+                </xacro:if>
+                <xacro:if value="${attachment == 'northrop_arm'}">
+                  <param name="gear_ratio">1.0</param>
+                </xacro:if>
                 <command_interface name="position"/>
                 <command_interface name="velocity"/>
@@ -68,5 +93,10 @@
             <joint name="rover_arm_wrist_roll_joint">
                 <param name="node_id">5</param>
-                <param name="gear_ratio">100.0</param>
+                <xacro:if value="${attachment == 'arm'}">
+                  <param name="gear_ratio">100.0</param>
+                </xacro:if>
+                <xacro:if value="${attachment == 'northrop_arm'}">
+                  <param name="gear_ratio">1.0</param>
+                </xacro:if>
                 <command_interface name="position"/>
                 <command_interface name="velocity"/>

File: software/ros_packages/rover2_arm/config/rover.urdf.xacro (robot description, xacro)
@@ -17,4 +17,7 @@
         <xacro:rover_ros2_control name="rover_arm" initial_positions_file="$(arg initial_positions_file)" ros2_control_hardware_type="$(arg ros2_control_hardware_type)"/>
     </xacro:if>
+    <xacro:if value="${front_attachment == 'northrop_arm'}">
+        <xacro:rover_ros2_control name="rover_arm" initial_positions_file="$(arg initial_positions_file)" ros2_control_hardware_type="$(arg ros2_control_hardware_type)"/>
+    </xacro:if>
     <!-- Include rover drive ros2_control -->
     <xacro:rover_body_ros2_control name="rover_drive" initial_positions_file="$(arg drive_initial_positions_file)" ros2_control_hardware_type="$(arg ros2_control_hardware_type)"/>

File: software/ros_packages/rover_urdf/urdf/rover2_urdf.xacro (robot description, xacro)
@@ -17,4 +17,17 @@
                 <origin rpy= "0.0 0.0 0.0" xyz="0.173803 -0.020767 0.071924"/>
             </xacro:rover2_arm>
+            <!-- Include sensors and other links -->
+            <xacro:include filename="$(find realsense2_description)/urdf/_d405.urdf.xacro"/>
+            <!-- Instantiate micros  -->
+            <xacro:sensor_d405 parent ="rover_arm_gripper" name="d405" use_nominal_extrinsics="true">
+                <!-- For older urdf <origin xyz="0 0.04075 0.1" rpy="0 -1.3963 -1.5708"/> -->
+                <origin xyz="-0.001611 -0.040711 0.099525" rpy="0.0 -1.3963635 1.5707963"/>
+            </xacro:sensor_d405>
+        </xacro:if>
+        <xacro:if value="${attachment== 'northrop_arm'}">
+            <xacro:include filename="$(find rover_arm_urdf)/urdf/northrop_arm.urdf.xacro" />
+            <xacro:northrop_arm parent="rover_base_origin" >
+                <origin rpy= "0.0 0.0 3.14159265359" xyz="0.231803 -0.020767 0.141924"/>
+            </xacro:northrop_arm>
             <!-- Include sensors and other links -->
             <xacro:include filename="$(find realsense2_description)/urdf/_d405.urdf.xacro"/>
